Commit message: 完成了机器人仿真模型的构建和显示功能，现在可以在RViz中查看SeaWashr机器人的3D模型。

File: Software/SeaWashr-ros2-ws/src/seaweashr-description/URDF/urdf/URDF.urdf (robot description, URDF)
Before this commit: robot URDF, 7 links, 6 joints
Links:
- added link world
- link base_link: geometry collision mesh filename=file:///home/tse-yatsing/Underwater_Cleaning_Robot/Software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; visual mesh filename=file:///home/tse-yatsing/Underwater_Cleaning_Robot/Software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
- link leftbackwheel_Link: geometry collision mesh filename=file:///home/tse-yatsing/Underwater_Cleaning_Robot/Software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; visual mesh filename=file:///home/tse-yatsing/Underwater_Cleaning_Robot/Software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
- link leftfrontwheel_Link: geometry collision mesh filename=file:///home/tse-yatsing/Underwater_Cleaning_Robot/Software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; visual mesh filename=file:///home/tse-yatsing/Underwater_Cleaning_Robot/Software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
- link leftmotor_Link: geometry collision mesh filename=file:///home/tse-yatsing/Underwater_Cleaning_Robot/Software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; visual mesh filename=file:///home/tse-yatsing/Underwater_Cleaning_Robot/Software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
- link rightbackwheel_Link: geometry collision mesh filename=file:///home/tse-yatsing/Underwater_Cleaning_Robot/Software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; visual mesh filename=file:///home/tse-yatsing/Underwater_Cleaning_Robot/Software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
- link rightfrontwheel_Link: geometry collision mesh filename=file:///home/tse-yatsing/Underwater_Cleaning_Robot/Software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; visual mesh filename=file:///home/tse-yatsing/Underwater_Cleaning_Robot/Software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
- link rightmotor_Link: geometry collision mesh filename=file:///home/tse-yatsing/Underwater_Cleaning_Robot/Software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; visual mesh filename=file:///home/tse-yatsing/Underwater_Cleaning_Robot/Software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
Joints:
- added joint world_to_base: type fixed, parent world, child base_link, origin xyz=0 0 0 rpy=-1.5708 0 0
- joint leftbackjoint: axis 0 0 0 -> 1 0 0
- joint leftfrontjoint: axis 0 0 0 -> 1 0 0
- joint leftmotorjoint: axis 0 0 0 -> 0 0 1
- joint rightbackjoint: axis 0 0 0 -> 1 0 0
- joint rightfrontjoint: axis 0 0 0 -> 1 0 0
- joint rightmotorjoint: axis 0 0 0 -> 0 0 1

Commit message: URDF.urdf改成相对路径

File: Software/SeaWashr-ros2-ws/src/seaweashr-description/URDF/urdf/URDF.urdf (robot description, URDF)
Before this commit: robot URDF, 8 links, 7 joints
Links:
- link base_link: geometry collision mesh filename=package://seaweashr-description/URDF/meshes/base_link.STL; visual mesh filename=package://seaweashr-description/URDF/meshes/base_link.STL
- link leftbackwheel_Link: geometry collision mesh filename=package://seaweashr-description/URDF/meshes/leftbackwheel_L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; visual mesh filename=package://seaweashr-description/URDF/meshes/leftbackwheel_L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
- link leftfrontwheel_Link: geometry collision mesh filename=package://seaweashr-description/URDF/meshes/leftfrontwheel_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; visual mesh filename=package://seaweashr-description/URDF/meshes/leftfrontwheel_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
- link leftmotor_Link: geometry collision mesh filename=package://seaweashr-description/URDF/meshes/leftmotor_Link.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; visual mesh filename=package://seaweashr-description/URDF/meshes/leftmotor_Link.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
- link rightbackwheel_Link: geometry collision mesh filename=package://seaweashr-description/URDF/meshes/rightbackwheel_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; visual mesh filename=package://seaweashr-description/URDF/meshes/rightbackwheel_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
- link rightfrontwheel_Link: geometry collision mesh filename=package://seaweashr-description/URDF/meshes/rightfrontwheel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; visual mesh filename=package://seaweashr-description/URDF/meshes/rightfrontwheel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
- link rightmotor_Link: geometry collision mesh filename=package://seaweashr-description/URDF/meshes/rightmotor_Link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; visual mesh filename=file:///home/tse-yatsing/Underwater_Cleaning_Robot/Software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
